File: Adafruit SMT Datalogger Shield rev C.brd (EAGLE design)
At the start: 68.6 x 53.3 mm, 44 parts, among them CN1 1X4-CLEANBIG, IC1 PCF8523T, M1 ARDUINO_R3_ICSP_NODIM, U2 4050, U3 MIC5225-3.3, Y1 32.768kHz

Commit message: fixval
Parts:
- R8: value 1k -> 10K
Changed lines of the file:
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@@
 <?xml version="1.0" encoding="utf-8"?>
 <!DOCTYPE eagle SYSTEM "eagle.dtd">
-<eagle version="9.0.1">
+<eagle version="9.1.3">
 <drawing>
 <settings>
-<setting alwaysvectorfont="no"/>
+<setting alwaysvectorfont="yes"/>
 <setting keepoldvectorfont="yes"/>
 <setting verticaltext="up"/>
@@
 <param name="checkStop" value="0"/>
 <param name="checkValues" value="0"/>
+<param name="checkNames" value="1"/>
+<param name="checkWireStubs" value="1"/>
+<param name="checkPolygonWidth" value="0"/>
 <param name="useDiameter" value="13"/>
 <param name="maxErrors" value="50"/>
@@
 <attribute name="VALUE" x="27.051" y="10.541" size="1.016" layer="27" ratio="10" rot="R180"/>
 </element>
-<element name="R8" library="microbuilder" package="0805-NO" value="1k" x="28.575" y="12.319" smashed="yes" rot="R180">
+<element name="R8" library="microbuilder" package="0805-NO" value="10K" x="28.575" y="12.319" smashed="yes" rot="R180">
 <attribute name="NAME" x="26.543" y="12.446" size="0.8128" layer="25" ratio="18" rot="R180"/>
 <attribute name="VALUE" x="26.543" y="13.335" size="1.016" layer="27" ratio="10"/>
@@
 </signal>
 </signals>
+<mfgpreviewcolors>
+<mfgpreviewcolor name="soldermaskcolor" color="0xC8008000"/>
+<mfgpreviewcolor name="silkscreencolor" color="0xFFFEFEFE"/>
+<mfgpreviewcolor name="backgroundcolor" color="0xFF282828"/>
+<mfgpreviewcolor name="coppercolor" color="0xFFFFBF00"/>
+<mfgpreviewcolor name="substratecolor" color="0xFF786E46"/>
+</mfgpreviewcolors>
 <errors>
 </errors>
