File: Adafruit SMT Datalogger Shield rev C.sch (EAGLE design)
At the start: 41 parts, among them CN1 1X4-CLEANBIG, IC1 PCF8523T, M1 ARDUINO_R3_ICSP_NODIM, U2 4050, U3 MIC5225-3.3, Y1 32.768kHz

Commit message: fixval
Parts:
- R8: value 1k -> 10K
Changed lines of the file:
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@@
 <?xml version="1.0" encoding="utf-8"?>
 <!DOCTYPE eagle SYSTEM "eagle.dtd">
-<eagle version="9.0.1">
+<eagle version="9.1.3">
 <drawing>
 <settings>
-<setting alwaysvectorfont="no"/>
+<setting alwaysvectorfont="yes"/>
 <setting keepoldvectorfont="yes"/>
 <setting verticaltext="up"/>
@@
 <part name="U$8" library="microbuilder" deviceset="VDDIO" device=""/>
 <part name="C1" library="microbuilder" deviceset="CAP_CERAMIC" device="0805-NOOUTLINE" value="10uF"/>
-<part name="R8" library="microbuilder" deviceset="RESISTOR" device="0805_NOOUTLINE" value="1k"/>
+<part name="R8" library="microbuilder" deviceset="RESISTOR" device="0805_NOOUTLINE" value="10K"/>
 <part name="U$9" library="microbuilder" deviceset="VDDIO" device=""/>
 <part name="GND14" library="supply1" deviceset="GND" device=""/>
